File: lizard.kicad_pcb (KiCad board)
At the start: 2 copper layers, 22 x 90 mm, 18 parts, among them P1 SWD, U1 EFM8BB1

Commit message: fixed bugs; added plots
Parts:
- added REF**: MountingHole_2-5mm, Mounting_Holes:MountingHole_2-5mm, F.Cu at (155.0, 155.0)
- added REF**: MountingHole_2-5mm, Mounting_Holes:MountingHole_2-5mm, F.Cu at (139.0, 155.0)
- added REF**: MountingHole_2-5mm, Mounting_Holes:MountingHole_2-5mm, F.Cu at (155.0, 113.0)
- added REF**: MountingHole_2-5mm, Mounting_Holes:MountingHole_2-5mm, F.Cu at (139.0, 113.0)
- added REF**: MountingHole_2-5mm, Mounting_Holes:MountingHole_2-5mm, F.Cu at (147.0, 65.0)
- moved BT1 8.00 mm to (147.1, 86.0)
- moved C1 8.00 mm to (140.5, 118.5)
- moved C2 8.00 mm to (140.5, 123.0)
- moved C3 8.00 mm to (147.5, 122.9)
- moved C4 8.00 mm to (153.5, 132.5)
- moved C5 8.00 mm to (153.5, 137.0)
- moved D1 8.00 mm to (144.3, 151.1)
- moved D2 8.00 mm to (150.1, 150.9)
- moved P1 8.00 mm to (140.5, 136.5)
- moved R1 8.00 mm to (152.5, 142.5)
- moved R2 8.00 mm to (140.5, 142.5)
- moved R3 8.00 mm to (148.5, 142.5)
- moved R4 8.00 mm to (144.5, 142.5)
- moved R5 8.00 mm to (153.9, 119.6)
- moved R6 8.00 mm to (147.5, 118.5)
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Other:
- board size 22 x 90 mm -> 22 x 98 mm
